File: Test Snubber/Test Snubber/Test Snubber.kicad_sch (KiCad schematic)
At the start: 21 parts, among them J1 1702473, J2 1702473, U1 AP63357QZV-7

Commit message: Finishes Test Snubber board
Parts:
- removed C11: EEE-1VA470WP, footprints:CAPAE660X580L260X65N, symbol capacitors:EEE-1VA470WP
- removed J2: 1702473, footprints:1702473, symbol connectors:_GENERIC_CONNECTOR_01x02
- added JP2: Jumper_NO_Small, Connector_PinHeader_2.54mm:PinHeader_1x02_P2.54mm_Vertical, symbol misc:Jumper_NO_Small
- added Q1: SI1442DH-T1-GE3, footprints:SOT23-6P95_285X140L45X42N, symbol mosfets:SI1442DH-T1-GE3
- added R6: 35028R2JT, footprints:RESISTOR_2010N, symbol resistors:35028R2JT
- renumbered R5 to R1, R1 to R2, R2 to R3, R3 to R4, R4 to R5
Connections:
- net +5V: now also R6.1
- net GND: now also JP2.1, Q1.4 (S)
- new net: Q1.1 (D), Q1.2 (D), Q1.5 (D), Q1.6 (D), R6.2
- new net: JP2.2, Q1.3 (G)
Other:
- note added: "@0.25A output current, 20mV input ripple, and 0.6A transient output: Inductance: 6.80uH Inductor ripple current: 1.29A Peak inductor current: 0.90A Peak input current: 0.06A RMS inductor current: 0.45A Total inductor energy: 2.73uJ Minimum ceramic input capacitance : 4.59uF Input transient current: 0.14A Minimum bulk input capacitance: 58.35uF Output ripple: 0.71mV"
- note removed: "@0.25A output current, 20mV input ripple, and 0.5A transient output: Inductance: 6.80uH Inductor ripple current: 1.29A Peak inductor current: 0.90A Peak input current: 0.06A RMS inductor current: 0.45A Total inductor energy: 2.73uJ Minimum ceramic input capacitance : 4.59uF Input transient current: 0.12A Minimum bulk input capacitance: 40.52uF Output ripple: 0.71mV"
