File: Test Snubber/Test Snubber/panel/Test Snubber Panel.kicad_pcb (KiCad board)
At the start: 2 copper layers, 67.9 x 45 mm, 29 parts, among them J1 1702473, Q1 SI1442DH-T1-GE3, U1 AP63357QZV-7

Commit message: Increases snubber panel size for PCBWay
Parts:
- removed the REF** at (30.0, 52.0) (x2)
- removed the REF** at (67.9, 23.0) (x2)
- removed the REF** at (30.0, 23.0) (x2)
- added REF**: Fiducial, Fiducial, F.Cu at (67.9, 23.0)
- added REF**: Fiducial, Fiducial, F.Cu at (30.0, 23.0)
- added REF**: Fiducial, Fiducial, F.Cu at (30.0, 67.0)
- added REF**: Fiducial, Fiducial, B.Cu at (30.0, 23.0)
- added REF**: Fiducial, Fiducial, B.Cu at (67.9, 23.0)
- added REF**: Fiducial, Fiducial, B.Cu at (30.0, 67.0)
- moved C1 7.50 mm to (42.5, 46.5)
- moved C10 7.50 mm to (58.0, 39.7)
- moved C2 7.50 mm to (53.4, 39.7)
- moved C3 7.50 mm to (49.3, 42.2)
- moved C4 7.50 mm to (52.7, 42.1)
- moved C5 7.50 mm to (52.7, 43.7)
- moved C6 7.50 mm to (52.7, 50.1)
- moved C7 7.50 mm to (57.2, 50.1)
- moved C8 7.50 mm to (50.3, 48.3)
- moved C9 7.50 mm to (57.0, 42.9)
- moved J1 7.50 mm to (33.2, 45.4)
- moved JP1 7.50 mm to (65.2, 49.5)
- moved JP2 7.50 mm to (70.1, 44.3)
- moved L1 7.50 mm to (56.9, 46.5)
- moved Q1 7.50 mm to (66.3, 45.7)
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Other:
- board size 67.9 x 45 mm -> 67.9 x 60 mm
